Commit message: JTC works for both arms and grippers

File: franka_description/robots/common/franka_arm.ros2_control.xacro (robot description, xacro)
@@ -4,11 +4,11 @@
          params="arm_id
              robot_ip
-             use_fake_hardware:=^|false
-             fake_sensor_commands:=^|false
+             use_fake_hardware:=^|true
+             fake_sensor_commands:=^|true
              gazebo:=^|false
-             hand:=^|false
+             hand:=^|true
              gazebo_effort:=^|false
              arm_prefix:=''
-             multi_arm:=false">
+             multi_arm:=true">
     <xacro:property name="arm_prefix_modified" value="${'' if arm_prefix == '' else arm_prefix + '_'}" />
     <ros2_control name="${arm_prefix_modified}FrankaHardwareInterface" type="system">
@@ -35,24 +35,20 @@
           </xacro:if>
         </hardware>
-      <xacro:macro name="configure_joint" params="joint_name initial_position">
+     <xacro:macro name="configure_joint" params="joint_name initial_position">
         <joint name="${joint_name}">
-          <!--
-            deactivated for gazebo velocity and position interface due to a bug
-            https://github.com/ros-controls/gz_ros2_control/issues/343
-            Command Interfaces -->
-          <xacro:if value="${multi_arm == 0}">
-            <command_interface name="position"/>
-            <command_interface name="velocity"/>
-          </xacro:if>
-          <xacro:if value="${gazebo == 0 or gazebo_effort == 1}">
-            <command_interface name="effort"/>
-          </xacro:if>
+          <!-- Command Interfaces -->
+          <command_interface name="position"/>
+          <command_interface name="velocity"/>
+          <command_interface name="effort"/>
           <!-- State Interfaces -->
           <state_interface name="position">
             <param name="initial_value">${initial_position}</param>
           </state_interface>
-          <state_interface name="velocity"/>
+          <state_interface name="velocity">
             <param name="initial_value">0.0</param>
-          <state_interface name="effort"/>
+          </state_interface>
+          <state_interface name="effort">
+            <param name="initial_value">0.0</param>
+          </state_interface>
         </joint>
       </xacro:macro>
@@ -64,6 +60,9 @@
       <xacro:configure_joint joint_name="${arm_prefix_modified}${arm_id}_joint6" initial_position="${pi/2}"/>
       <xacro:configure_joint joint_name="${arm_prefix_modified}${arm_id}_joint7" initial_position="${pi/4}"/>
+      <!-- Left gripper joints -->
+      <xacro:configure_joint joint_name="${arm_prefix_modified}${arm_id}_finger_joint1" initial_position="0.039"/>
+      <xacro:configure_joint joint_name="${arm_prefix_modified}${arm_id}_finger_joint2" initial_position="0.039"/>
       <xacro:if value="${gazebo and hand}">
-        <xacro:configure_joint joint_name="${arm_id}_finger_joint1" initial_position="0.0" />
+        <xacro:configure_joint joint_name="${arm_id}_finger_joint1" initial_position="0.039" />
       </xacro:if>
     </ros2_control>

File: franka_description/robots/common/franka_robot.xacro (robot description, xacro)
@@ -16,6 +16,6 @@
                       ros2_control:=false
                       robot_ip:=''
-                      use_fake_hardware:=false
-                      fake_sensor_commands:=false
+                      use_fake_hardware:=true
+                      fake_sensor_commands:=true
                       gazebo_effort:=false
                       no_prefix:='false'

File: franka_description/robots/multi_arm/multi_arm.urdf.xacro (robot description, xacro)
@@ -12,5 +12,5 @@
   <xacro:arg name="number_of_robots" default = "2"/>
   <!-- Define arguments -->
-  <xacro:arg name="xyz_values" default="['0 0.7 0','0 -0.7 0']" />
+  <xacro:arg name="xyz_values" default="['0 0.75 0','0 -0.75 0']" />
   <xacro:property name="xyz_list" value="${$(arg xyz_values)}" />
   <!-- Define arguments -->
@@ -26,12 +26,12 @@
   <xacro:arg name="with_sc" default="false" />
   <!-- Is the robot being controlled with ros2_control?" -->
-  <xacro:arg name="ros2_control" default="false" />
+  <xacro:arg name="ros2_control" default="true" />
   <!-- IP address or hostname of the robot" -->
   <xacro:arg name="robot_ips" default="['172.16.0.2','172.16.0.3']" />
   <xacro:property name="robot_ips_list" value="${$(arg robot_ips)}" />
   <!-- Should a fake hardware be used? -->
-  <xacro:arg name="use_fake_hardware" default="false" />
+  <xacro:arg name="use_fake_hardware" default="true" />
   <!-- Should fake sensors be used? -->
-  <xacro:arg name="fake_sensor_commands" default="false" />
+  <xacro:arg name="fake_sensor_commands" default="true" />
   <!-- Should the robot be spawned in Gazebo?" -->
   <xacro:arg name="gazebo" default="false" />
